File: pcb/Prototype1.brd (EAGLE design)
At the start: 37.8 x 38.1 mm, 30 parts, among them IC1 78L05SMD, Q1 FDS5680, U1 PIC16F1823-X_SL

Commit message: Added waveforms, added component values to schematic. Added fail description, and lesson learned to readme.
Parts:
- C1, C2, C3: value (none) -> 47u
- C4: value (none) -> 100n
- R1: value (none) -> 47
- R2, R3: value (none) -> 2.2k
- R4: value (none) -> 100k
- R5: value (none) -> 180k
- R6, R7: value (none) -> 680
Changed lines of the file:
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@@
 </autorouter>
 <elements>
-<element name="C1" library="rcl" package="153CLV-0605" value="" x="7.62" y="16.51" smashed="yes">
+<element name="C1" library="rcl" package="153CLV-0605" value="47u" x="7.62" y="16.51" smashed="yes">
 <attribute name="NAME" x="1.69" y="18.87" size="1.27" layer="25"/>
 <attribute name="VALUE" x="4.195" y="11.625" size="1.27" layer="27"/>
 </element>
-<element name="C2" library="rcl" package="153CLV-0605" value="" x="7.62" y="24.13" smashed="yes">
+<element name="C2" library="rcl" package="153CLV-0605" value="47u" x="7.62" y="24.13" smashed="yes">
 <attribute name="NAME" x="1.69" y="26.49" size="1.27" layer="25"/>
 <attribute name="VALUE" x="4.195" y="19.245" size="1.27" layer="27"/>
 </element>
-<element name="C3" library="rcl" package="153CLV-0605" value="" x="7.62" y="31.75" smashed="yes">
+<element name="C3" library="rcl" package="153CLV-0605" value="47u" x="7.62" y="31.75" smashed="yes">
 <attribute name="NAME" x="1.69" y="32.84" size="1.27" layer="25"/>
 <attribute name="VALUE" x="4.195" y="26.865" size="1.27" layer="27"/>
 </element>
-<element name="C4" library="rcl" package="C0805" value="" x="21.59" y="17.78" rot="R90"/>
+<element name="C4" library="rcl" package="C0805" value="100n" x="21.59" y="17.78" rot="R90"/>
 <element name="D1" library="diode" package="MELF-MLL41" value="" x="13.97" y="11.43" smashed="yes" rot="R180">
 <attribute name="NAME" x="12.188" y="14.151" size="1.27" layer="25" rot="R180"/>
@@
 </element>
 <element name="Q1" library="transistor-fet" package="SO-8" value="FDS5680" x="30.48" y="5.08" rot="R180"/>
-<element name="R1" library="rcl" package="M1206" value="" x="30.48" y="10.16"/>
-<element name="R2" library="rcl" package="M1206" value="" x="1.905" y="10.16" smashed="yes" rot="R90">
+<element name="R1" library="rcl" package="M1206" value="47" x="30.48" y="10.16"/>
+<element name="R2" library="rcl" package="M1206" value="2.2k" x="1.905" y="10.16" smashed="yes" rot="R90">
 <attribute name="NAME" x="1.905" y="15.24" size="1.27" layer="25" rot="R90"/>
 <attribute name="VALUE" x="4.445" y="8.89" size="1.27" layer="27" rot="R90"/>
 </element>
-<element name="R3" library="rcl" package="M1206" value="" x="5.08" y="10.16" smashed="yes" rot="R90">
+<element name="R3" library="rcl" package="M1206" value="2.2k" x="5.08" y="10.16" smashed="yes" rot="R90">
 <attribute name="NAME" x="6.35" y="11.43" size="1.27" layer="25" rot="R270"/>
 <attribute name="VALUE" x="7.62" y="8.89" size="1.27" layer="27" rot="R90"/>
 </element>
-<element name="R4" library="rcl" package="M1206" value="" x="25.4" y="10.16"/>
-<element name="R5" library="rcl" package="M1206" value="" x="24.13" y="5.08" rot="R270"/>
-<element name="R6" library="rcl" package="M1206" value="" x="33.02" y="29.21" rot="R270"/>
-<element name="R7" library="rcl" package="M1206" value="" x="29.21" y="29.21" rot="R270"/>
+<element name="R4" library="rcl" package="M1206" value="100k" x="25.4" y="10.16"/>
+<element name="R5" library="rcl" package="M1206" value="180k" x="24.13" y="5.08" rot="R270"/>
+<element name="R6" library="rcl" package="M1206" value="680" x="33.02" y="29.21" rot="R270"/>
+<element name="R7" library="rcl" package="M1206" value="680" x="29.21" y="29.21" rot="R270"/>
 <element name="SV1" library="con-lsta" package="FE05-1" value="" x="19.05" y="34.29">
 <attribute name="MF" value="" x="19.05" y="34.29" size="1.778" layer="27" display="off"/>
